File: bbhTiny84.sch (EAGLE design)
At the start: 13 parts, among them U1 ATtinyX4

Commit message: Add board and schematic images.
Other:
- note added: "v1"
Changed lines of the file:
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@@
 under CC BY-SA 4.0 http://creativecommons.org/licenses/by-sa/4.0/                       </text>
 <text x="15.24" y="27.94" size="3.81" layer="94" ratio="12">CC BY-SA</text>
+<text x="264.16" y="7.62" size="2.54" layer="94" ratio="12">v1</text>
 </plain>
 <instances>
